File: hardware/displays/IN-12/IN-12.kicad_pcb (KiCad board)
At the start: 2 copper layers, 150 x 52 mm, 48 parts, among them J1 Conn_02x06_Odd_Even, J2 Conn_01x06, J3 Conn_02x06_Odd_Even, T1 IN-12B_Nixie_Tube, T2 IN-12B_Nixie_Tube, T3 IN-12B_Nixie_Tube, T4 IN-12B_Nixie_Tube, T5 IN-12B_Nixie_Tube, T6 IN-12B_Nixie_Tube, U1 CD40109B, U2 HV5622, U3 HV5622, U4 HV5622

Commit message: Latest changes in ToT, might not want all of these
Connections:
- net ~BL_DB~ renamed ~{BL_DB}
- net ~BL~ renamed ~{BL}
- net ~LE_DB~ renamed ~{LE_DB}
- net ~LE~ renamed ~{LE}
Other:
- net class Default removed
- net class HV removed
- net class Power removed
