File: hardware/logic/v1/TubeClock-2Layer.kicad_pcb (KiCad board)
At the start: 2 copper layers, 150 x 70 mm, 147 parts, among them J1 Jack-DC, J2 Conn_02x08_Odd_Even, J3 Conn_02x05_Odd_Even, J4 Conn_02x06_Odd_Even, J5 Conn_01x06, J6 Conn_02x03_Odd_Even, J7 Conn_01x07, J8 Conn_Coaxial, P1 STM32_SWD_USART, P2 CONN_MICRO_USB_B, Q1 IRF644PBF, Q2 Q_Photo_NPN, Q3 2N7002, Q4 2N7002, Q5 2N7002, Q6 2N7002, SW1 SW_Push, SW2 SW_Push, U1 MAX1771, U10 Teseo-LIV3F, U11 TPS22943, U2 LD1117S33TR, U3 STM32F072RBTx, U4 TSOP382xx, U5 DS3234, U6 LM74, U7 DS1722, U8 MAX485E, U9 BGA824N6, Y1 8 MHz, Y2 32.768 KHz

Commit message: All latest produced changes
Parts:
- F1: value ~2A -> ~{2A}
Other:
- net class 12V removed
- net class 3V3 removed
- net class Default removed
- net class HV removed
- net class PowerIn removed
- net class Touchkey removed
- net class USB removed
